Commit message: fix: urdf -> xacro

File: vs050_description/vs050.urdf.xacro (robot description, xacro)
@@ -1,3 +1,4 @@
 <?xml version="1.0" encoding="UTF-8"?>
+<xacro:macro name="vs050" params="platform">
 <robot name="vs050">
 	<gazebo>
@@ -253,2 +254,3 @@
 	</transmission>
 </robot>
+</xacro:macro>
